File: board/Dilbert-Badge.brd (EAGLE design)
At the start: 101.3 x 48.2 mm, 31 parts, among them IC1 MCP23017SO, J5 I2C, J6 UART, J7 NEOPIXEL, SW1 UP, SW2 DOWN, SW3 LEFT, SW4 RIGHT, SW5 A, SW6 B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

Commit message: board updates
Parts:
- removed J6: UART, SparkFun-Connectors:1X06
- added J2: FTDI_DEVICE, SparkFun-Connectors:FTDI_DEVICE_SIDE
- added JP1, JP2, JP3: JUMPER-PAD-3-NOFULL_BOX_SILK, SparkFun-Passives:PAD-JUMPER-3-NO_YES_SILK_FULL_BOX
- added JP4, JP5: JUMPER-PAD-2-NC_BY_TRACENO_SILK, SparkFun-Passives:PAD-JUMPER-2-NC_BY_TRACE_NO_SILK
- added R4: 10K, adafruit:R0805
- moved SW5 89.6 mm to (94.0, 49.5)
- moved SW2 88.2 mm to (95.2, 21.6)
- moved SW3 78.2 mm to (90.2, 27.9)
- moved SW4 78.2 mm to (90.2, 15.2)
- moved SW6 72.4 mm to (86.4, 41.9)
- moved SW1 68.4 mm to (85.1, 21.6)
- moved X1 66.7 mm to (17.8, 19.1), turned to 270 degrees
- moved LED8 64.7 mm to (74.9, 53.3)
- moved LED1 61.1 mm to (74.9, 8.89)
- moved LED7 56.1 mm to (74.9, 47.0)
- moved LED2 53.2 mm to (74.9, 15.2)
- moved LED6 49.4 mm to (74.9, 40.6)
- moved LED3 47.4 mm to (74.9, 21.6)
- moved LED5 45.3 mm to (74.9, 34.3)
- moved J7 45.1 mm to (63.5, 53.3), turned to 180 degrees
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Connections:
- new net MCP_IO_A0: IC1.15, JP1.2
- new net MCP_IO_A1: IC1.16, JP2.2
- new net MCP_IO_A2: IC1.17, JP3.2
- new net MCP_IO_INT: IC1.20, JP4.2
- new net MCP_IO_RST: IC1.18, R4.1
- net 3V3: now also J2.P$4, JP1.3, JP2.3, JP3.3, R4.2; no longer J6.4
- net GND: now also J2.P$6, JP1.1, JP2.1, JP3.1; no longer J6.6
- net SD_CS: now also JP5.2
- net UART_CTS: now also J2.P$5; no longer J6.5
- net UART_DTR: now also J2.P$1; no longer J6.1
- net UART_RX: now also J2.P$3, JP5.1; no longer J6.3
- net UART_TX: now also J2.P$2, JP4.1; no longer J6.2
Other:
- board outline removed

Commit message: more board layout
Parts:
- removed J7: NEOPIXEL, connectors:3X1_SMD
- added J3: NEOPIXEL, SparkFun-Connectors:1X03
- added U$2, U$3: 5MM_MOUNTING_HOLE, mechanical:5MM_HOLE
- J1: value (none) -> IO EXP.; device connectors:10X1_SMD -> SparkFun-Connectors:1X10
- JP1: value JUMPER-PAD-3-NOFULL_BOX_SILK -> MCP IO A0; device SparkFun-Passives:PAD-JUMPER-3-NO_YES_SILK_FULL_BOX -> SparkFun-Passives:PAD-JUMPER-3-NO_YES_SILK
- JP2: value JUMPER-PAD-3-NOFULL_BOX_SILK -> MCP IO A1; device SparkFun-Passives:PAD-JUMPER-3-NO_YES_SILK_FULL_BOX -> SparkFun-Passives:PAD-JUMPER-3-NO_YES_SILK
- JP3: value JUMPER-PAD-3-NOFULL_BOX_SILK -> MCP IO A2; device SparkFun-Passives:PAD-JUMPER-3-NO_YES_SILK_FULL_BOX -> SparkFun-Passives:PAD-JUMPER-3-NO_YES_SILK
- JP4: value JUMPER-PAD-2-NC_BY_TRACENO_SILK -> IO INT TO UART TX
- JP5: value JUMPER-PAD-2-NC_BY_TRACENO_SILK -> SD CS TO UART RX
- moved LOGO1 69.0 mm to (99.7, 43.2), turned to 90 degrees
- moved JP3 63.4 mm to (59.7, 12.7), flipped to the bottom
- moved R4 60.2 mm to (62.2, 19.1), turned to 270 degrees
- moved JP2 57.5 mm to (55.9, 12.7), flipped to the bottom
- moved JP1 51.7 mm to (52.1, 12.7), flipped to the bottom
- moved R3 51.2 mm to (36.8, 19.1), turned to 270 degrees
- moved R6 50.2 mm to (33.0, 12.7), turned to 90 degrees
- moved R5 32.4 mm to (34.3, 48.3), turned to 270 degrees
- moved JP4 28.2 mm to (34.3, 21.6)
- moved R1 18.8 mm to (24.1, 48.3), turned to 270 degrees
- moved R2 16.7 mm to (17.8, 40.6), turned to 90 degrees
- moved JP5 14.5 mm to (11.4, 30.5), turned to 0 degrees
- moved J1 13.0 mm to (40.6, 39.4), flipped to the top
- moved C1 6.35 mm to (14.0, 64.8), turned to 270 degrees
- moved J5 5.08 mm to (48.3, 7.62), turned to 180 degrees
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Connections:
- net 3V3: now also J3.2; no longer J7.2
- net GND: now also J3.1; no longer J7.1
- net NEOPIXEL_OUT: now also J3.3; no longer J7.3
Routing:
- net TFT_CS: track 0.00 -> 106.2 mm, vias 0 -> 1
- net SCK: track 0.00 -> 79.0 mm, vias 0 -> 2
- net MISO: track 0.00 -> 78.0 mm, vias 0 -> 2
- net MOSI: track 0.00 -> 75.2 mm, vias 0 -> 2
- net TFT_BL: track 0.00 -> 58.4 mm, vias 0 -> 1
- net BTN_A: track 0.00 -> 48.2 mm, vias 0 -> 1
- net BTN_D: track 0.00 -> 39.4 mm
- net BTN_R: track 0.00 -> 36.0 mm
- net RESET: track 0.00 -> 36.0 mm
- net BTN_B: track 0.00 -> 33.1 mm, vias 0 -> 1
- net BTN_L: track 0.00 -> 31.8 mm
- net 3V3: track 0.00 -> 31.6 mm
- net N$8: track 0.00 -> 31.0 mm, vias 0 -> 1
- net BTN_U: track 0.00 -> 28.3 mm
- net N$9: track 0.00 -> 27.9 mm, vias 0 -> 1
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- added copper zone on layer 1, net 3V3
- added copper zone on layer 1, net GND
- added copper zone on layer 16, net GND
Other:
- board outline added: 105.4 x 52.1 mm
