File: board/Dilbert-Badge.sch (EAGLE design)
At the start: 27 parts, among them IC1 MCP23017SO, J1 I2C, J2 UART, J6 IO_B, J7 IO_A, SW1 UP, SW2 DOWN, SW3 LEFT, SW4 RIGHT, SW5 A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

Commit message: Update board
[ci skip]
Parts:
- added R5, R6: 10K, adafruit:R-US_R0805
- R4: value (none) -> 10K
Connections:
- net LED_OUT renamed NEOPIXEL_OUT
- net N$10 renamed MOSI
- net N$11 renamed MISO
- net N$12 renamed TFT_CS
- net N$9 renamed SCK
- removed net LED_IN: J5.7, LED1.DI, R4.2, X1.GPIO15
- new net NEOPIXEL: J5.7, LED1.DI, R6.2, X1.GPIO15
- new net TFT_DC: J5.6, R4.1, X1.GPIO2
- net 3V3: now also R4.2, R5.2
- net GND: now also R6.1; no longer R4.1
- net GPIO2: no longer J5.6, X1.GPIO2
- net SCL: now also R5.1
Changed lines of the file:
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@@
 <setting verticaltext="up"/>
 </settings>
-<grid distance="0.1" unitdist="inch" unit="inch" style="lines" multiple="1" display="yes" altdistance="0.01" altunitdist="inch" altunit="inch"/>
+<grid distance="0.1" unitdist="inch" unit="inch" style="lines" multiple="1" display="no" altdistance="0.01" altunitdist="inch" altunit="inch"/>
 <layers>
 <layer number="1" name="Top" color="4" fill="1" visible="no" active="no"/>
@@
 <part name="R2" library="adafruit" deviceset="R-US_" device="R0805" value="10K"/>
 <part name="R3" library="adafruit" deviceset="R-US_" device="R0805" value="10K"/>
-<part name="R4" library="adafruit" deviceset="R-US_" device="R0805"/>
+<part name="R4" library="adafruit" deviceset="R-US_" device="R0805" value="10K"/>
 <part name="C1" library="SparkFun-Capacitors" deviceset="10UF10V10%(0805)" device=""/>
+<part name="R5" library="adafruit" deviceset="R-US_" device="R0805" value="10K"/>
+<part name="R6" library="adafruit" deviceset="R-US_" device="R0805" value="10K"/>
 </parts>
 <sheets>
@@
 <instance part="R4" gate="G$1" x="193.04" y="144.78" rot="R90"/>
 <instance part="C1" gate="G$1" x="152.4" y="109.22"/>
+<instance part="R5" gate="G$1" x="132.08" y="160.02" rot="R90"/>
+<instance part="R6" gate="G$1" x="210.82" y="144.78" rot="R90"/>
 </instances>
 <busses>
@@
 </segment>
 <segment>
-<pinref part="R4" gate="G$1" pin="1"/>
-<wire x1="193.04" y1="134.62" x2="193.04" y2="139.7" width="0.1524" layer="91"/>
-<label x="193.04" y="134.62" size="1.778" layer="95" rot="MR180"/>
-</segment>
-<segment>
 <pinref part="C1" gate="G$1" pin="2"/>
 <wire x1="152.4" y1="106.68" x2="152.4" y2="101.6" width="0.1524" layer="91"/>
 <label x="152.4" y="101.6" size="1.778" layer="95" rot="MR180"/>
+</segment>
+<segment>
+<pinref part="R6" gate="G$1" pin="1"/>
+<wire x1="210.82" y1="139.7" x2="210.82" y2="134.62" width="0.1524" layer="91"/>
+<label x="210.82" y="134.62" size="1.778" layer="95" rot="MR180"/>
 </segment>
 </net>
@@
 <segment>
 <pinref part="SW8" gate="G$1" pin="P$2"/>
-<label x="132.08" y="154.94" size="1.778" layer="95"/>
-<wire x1="132.08" y1="154.94" x2="132.08" y2="149.86" width="0.1524" layer="91"/>
+<label x="137.16" y="152.4" size="1.778" layer="95"/>
+<wire x1="132.08" y1="154.94" x2="132.08" y2="152.4" width="0.1524" layer="91"/>
+<wire x1="132.08" y1="152.4" x2="132.08" y2="149.86" width="0.1524" layer="91"/>
+<wire x1="137.16" y1="152.4" x2="132.08" y2="152.4" width="0.1524" layer="91"/>
+<pinref part="R5" gate="G$1" pin="1"/>
 </segment>
 </net>
@@
 </segment>
 </net>
-<net name="LED_OUT" class="0">
+<net name="NEOPIXEL_OUT" class="0">
 <segment>
 <pinref part="LED4" gate="G$1" pin="DO"/>
@@
 </segment>
 </net>
-<net name="LED_IN" class="0">
+<net name="NEOPIXEL" class="0">
 <segment>
 <pinref part="LED1" gate="G$1" pin="DI"/>
@@
 </segment>
 <segment>
-<pinref part="R4" gate="G$1" pin="2"/>
-<wire x1="193.04" y1="154.94" x2="193.04" y2="149.86" width="0.1524" layer="91"/>
-<label x="193.04" y="154.94" size="1.778" layer="95"/>
+<pinref part="R6" gate="G$1" pin="2"/>
+<wire x1="210.82" y1="149.86" x2="210.82" y2="154.94" width="0.1524" layer="91"/>
+<label x="210.82" y="154.94" size="1.778" layer="95"/>
 </segment>
 </net>
@@
 </segment>
 </net>
-<net name="N$9" class="0">
+<net name="SCK" class="0">
 <segment>
 <pinref part="J4" gate="G$1" pin="4"/>
 <pinref part="X1" gate="G$1" pin="GPIO14"/>
 <wire x1="45.72" y1="71.12" x2="66.04" y2="71.12" width="0.1524" layer="91"/>
-</segment>
-</net>
-<net name="N$10" class="0">
+<label x="63.5" y="71.12" size="1.778" layer="95" rot="MR0"/>
+</segment>
+</net>
+<net name="MOSI" class="0">
 <segment>
 <pinref part="J4" gate="G$1" pin="2"/>
 <pinref part="X1" gate="G$1" pin="GPIO13"/>
 <wire x1="45.72" y1="66.04" x2="66.04" y2="66.04" width="0.1524" layer="91"/>
-</segment>
-</net>
-<net name="N$11" class="0">
+<label x="63.5" y="66.04" size="1.778" layer="95" rot="MR0"/>
+</segment>
+</net>
+<net name="MISO" class="0">
 <segment>
 <pinref part="X1" gate="G$1" pin="GPIO12"/>
 <pinref part="J4" gate="G$1" pin="3"/>
 <wire x1="66.04" y1="68.58" x2="45.72" y2="68.58" width="0.1524" layer="91"/>
-</segment>
-</net>
-<net name="N$12" class="0">
+<label x="63.5" y="68.58" size="1.778" layer="95" rot="MR0"/>
+</segment>
+</net>
+<net name="TFT_CS" class="0">
 <segment>
 <pinref part="X1" gate="G$1" pin="GPIO4"/>
 <pinref part="J5" gate="G$1" pin="3"/>
 <wire x1="101.6" y1="76.2" x2="121.92" y2="76.2" width="0.1524" layer="91"/>
+<label x="104.14" y="76.2" size="1.778" layer="95"/>
 </segment>
 </net>
 <net name="GPIO2" class="0">
-<segment>
-<pinref part="J5" gate="G$1" pin="6"/>
-<pinref part="X1" gate="G$1" pin="GPIO2"/>
-<wire x1="121.92" y1="68.58" x2="101.6" y2="68.58" width="0.1524" layer="91"/>
-<label x="104.14" y="68.58" size="1.778" layer="95"/>
-</segment>
 <segment>
 <pinref part="R3" gate="G$1" pin="1"/>
@@
 <label x="152.4" y="119.38" size="1.778" layer="95"/>
 </segment>
-</net>
+<segment>
+<pinref part="R5" gate="G$1" pin="2"/>
+<wire x1="132.08" y1="170.18" x2="132.08" y2="165.1" width="0.1524" layer="91"/>
+<label x="132.08" y="170.18" size="1.778" layer="95"/>
+</segment>
+<segment>
+<pinref part="R4" gate="G$1" pin="2"/>
+<wire x1="193.04" y1="154.94" x2="193.04" y2="149.86" width="0.1524" layer="91"/>
+<label x="193.04" y="154.94" size="1.778" layer="95"/>
+</segment>
+</net>
+<net name="TFT_DC" class="0">
+<segment>
+<pinref part="J5" gate="G$1" pin="6"/>
+<pinref part="X1" gate="G$1" pin="GPIO2"/>
+<wire x1="121.92" y1="68.58" x2="101.6" y2="68.58" width="0.1524" layer="91"/>
+<label x="104.14" y="68.58" size="1.778" layer="95"/>
+</segment>
+<segment>
+<pinref part="R4" gate="G$1" pin="1"/>
+<wire x1="193.04" y1="134.62" x2="193.04" y2="139.7" width="0.1524" layer="91"/>
+<label x="193.04" y="134.62" size="1.778" layer="95" rot="MR180"/>
+</segment>
+</net>

Commit message: More dev work
Connections:
- net N$7 renamed GPIO16
- net TFT_CS renamed GPIO4
- removed net TFT_DC: J5.6, R4.1, X1.GPIO2
- net GPIO2: now also J5.6, R4.1, X1.GPIO2
Changed lines of the file:
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@@
 </segment>
 </net>
-<net name="N$7" class="0">
+<net name="GPIO16" class="0">
 <segment>
 <pinref part="X1" gate="G$1" pin="GPIO16"/>
 <pinref part="J4" gate="G$1" pin="5"/>
 <wire x1="66.04" y1="73.66" x2="45.72" y2="73.66" width="0.1524" layer="91"/>
+<label x="63.5" y="73.66" size="1.778" layer="95" rot="MR0"/>
 </segment>
 </net>
@@
 </segment>
 </net>
-<net name="TFT_CS" class="0">
+<net name="GPIO4" class="0">
 <segment>
 <pinref part="X1" gate="G$1" pin="GPIO4"/>
@@
 <wire x1="175.26" y1="139.7" x2="175.26" y2="134.62" width="0.1524" layer="91"/>
 <label x="175.26" y="134.62" size="1.778" layer="95" rot="MR180"/>
+</segment>
+<segment>
+<pinref part="J5" gate="G$1" pin="6"/>
+<pinref part="X1" gate="G$1" pin="GPIO2"/>
+<wire x1="121.92" y1="68.58" x2="101.6" y2="68.58" width="0.1524" layer="91"/>
+<label x="104.14" y="68.58" size="1.778" layer="95"/>
+</segment>
+<segment>
+<pinref part="R4" gate="G$1" pin="1"/>
+<wire x1="193.04" y1="134.62" x2="193.04" y2="139.7" width="0.1524" layer="91"/>
+<label x="193.04" y="134.62" size="1.778" layer="95" rot="MR180"/>
 </segment>
 </net>
@@
 </segment>
 </net>
-<net name="TFT_DC" class="0">
-<segment>
-<pinref part="J5" gate="G$1" pin="6"/>
-<pinref part="X1" gate="G$1" pin="GPIO2"/>
-<wire x1="121.92" y1="68.58" x2="101.6" y2="68.58" width="0.1524" layer="91"/>
-<label x="104.14" y="68.58" size="1.778" layer="95"/>
-</segment>
-<segment>
-<pinref part="R4" gate="G$1" pin="1"/>
-<wire x1="193.04" y1="134.62" x2="193.04" y2="139.7" width="0.1524" layer="91"/>
-<label x="193.04" y="134.62" size="1.778" layer="95" rot="MR180"/>
-</segment>
-</net>

Commit message: more work on board
Parts:
- removed J2: UART, SparkFun-Connectors:M06SILK_FEMALE_PTH
- removed J3: (no value), SparkFun-Connectors:M03PTH
- removed J4: (no value), SparkFun-Connectors:M08NO_SILK_FEMALE_PTH
- added R7: 10K, adafruit:R-US_R0805
- added U$1: 2.2IN_ILI9341, displays:2.2IN_ILI9341
- J1: value I2C -> (none); device SparkFun-Connectors:M04PTH -> connectors:10X1_SMD_HEADER
- J5: value (none) -> I2C; device SparkFun-Connectors:M08NO_SILK_FEMALE_PTH -> SparkFun-Connectors:M04PTH
- J6: value IO_B -> UART; device SparkFun-Connectors:M08 -> SparkFun-Connectors:M06SILK_FEMALE_PTH
- J7: value IO_A -> NEOPIXEL; device SparkFun-Connectors:M08 -> connectors:3X1_SMD_HEADER
Connections:
- removed net N$14: IC1.GPB0, J6.1
- removed net N$15: IC1.GPB1, J6.2
- removed net N$16: IC1.GPB7, J6.8
- removed net N$17: IC1.GPB6, J6.7
- removed net N$18: IC1.GPB5, J6.6
- removed net N$19: IC1.GPB4, J6.5
- removed net N$20: IC1.GPB3, J6.4
- removed net N$21: IC1.GPB2, J6.3
- removed net N$22: IC1.GPA7, J7.8
- removed net N$23: IC1.GPA6, J7.7
- new net N$10: IC1.GPB7, J1.8
- new net N$11: IC1.GPB6, J1.7
- new net N$12: IC1.GPB5, J1.6
- new net N$13: IC1.GPB4, J1.5
- new net N$4: IC1.GPB0, J1.1
- new net N$5: IC1.GPB1, J1.2
- new net N$6: IC1.GPB2, J1.3
- new net N$7: IC1.GPB3, J1.4
- new net N$8: IC1.GPA7, J1.10
- new net N$9: IC1.GPA6, J1.9
- new net SD_CS: U$1.SD_CS
- new net TFT_BL: U$1.LED
- new net TFT_CS: U$1.CS
- new net TFT_DC: U$1.DC
- new net TFT_RESET: R7.1, U$1.RESET
- net 3V3: now also J5.2, J6.4, J7.2, R7.2, U$1.VCC; no longer J1.2, J2.4, J3.2, J4.1
- net BTN_A: no longer J7.5
- net BTN_B: no longer J7.6
- net BTN_D: no longer J7.2
- net BTN_L: no longer J7.3
- net BTN_R: no longer J7.4
- net BTN_U: no longer J7.1
- net ESP_ADC: no longer J4.7
- net ESP_CH_PD: no longer J4.6
- net GND: now also J5.1, J6.6, J7.1, U$1.GND; no longer J1.1, J2.6, J3.1, J5.8
- net GPIO16: no longer J4.5
- net GPIO2: no longer J5.6
- net GPIO4: no longer J5.3
- net MISO: now also U$1.MISO, U$1.SD_MISO; no longer J4.3
- net MOSI: now also U$1.MOSI, U$1.SD_MOSI; no longer J4.2
- net NEOPIXEL: no longer J5.7
- net NEOPIXEL_OUT: now also J7.3; no longer J3.3
- net RESET: no longer J4.8
- net SCK: now also U$1.SCK, U$1.SD_SCK; no longer J4.4
- net SCL: now also J5.4; no longer J1.4, J5.5
- net SDA: now also J5.3; no longer J1.3, J5.4
- net UART_CTS: now also J6.5; no longer J2.5
- net UART_DTR: now also J6.1; no longer J2.1
- net UART_RX: now also J6.3; no longer J2.3, J5.2
- net UART_TX: now also J6.2; no longer J2.2, J5.1

Commit message: more work
Connections:
- removed net GPIO16: X1.GPIO16
- removed net GPIO4: X1.GPIO4
- new net GPIO0: R5.1, SW8.P$2, X1.GPIO0
- net SCL: now also X1.GPIO5; no longer R5.1, SW8.P$2, X1.GPIO0
- net SDA: now also X1.GPIO4; no longer X1.GPIO5
- net TFT_BL: now also X1.GPIO16
Changed lines of the file:
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@@
 <setting verticaltext="up"/>
 </settings>
-<grid distance="0.1" unitdist="inch" unit="inch" style="lines" multiple="1" display="yes" altdistance="0.01" altunitdist="inch" altunit="inch"/>
+<grid distance="0.1" unitdist="inch" unit="inch" style="lines" multiple="1" display="no" altdistance="0.01" altunitdist="inch" altunit="inch"/>
 <layers>
 <layer number="1" name="Top" color="4" fill="1" visible="no" active="no"/>
@@
 <net name="SDA" class="0">
 <segment>
+<wire x1="83.82" y1="111.76" x2="81.28" y2="111.76" width="0.1524" layer="91"/>
+<label x="83.82" y="111.76" size="1.778" layer="95"/>
+<pinref part="J5" gate="G$1" pin="3"/>
+</segment>
+<segment>
+<pinref part="IC1" gate="G$1" pin="SDA"/>
+<wire x1="185.42" y1="43.18" x2="187.96" y2="43.18" width="0.1524" layer="91"/>
+<label x="185.42" y="43.18" size="1.778" layer="95" rot="MR0"/>
+</segment>
+<segment>
+<pinref part="X1" gate="G$1" pin="GPIO4"/>
+<wire x1="101.6" y1="76.2" x2="121.92" y2="76.2" width="0.1524" layer="91"/>
+<label x="104.14" y="76.2" size="1.778" layer="95"/>
+</segment>
+</net>
+<net name="SCL" class="0">
+<segment>
+<wire x1="83.82" y1="114.3" x2="81.28" y2="114.3" width="0.1524" layer="91"/>
+<label x="83.82" y="114.3" size="1.778" layer="95"/>
+<pinref part="J5" gate="G$1" pin="4"/>
+</segment>
+<segment>
+<pinref part="IC1" gate="G$1" pin="SCL"/>
+<wire x1="185.42" y1="45.72" x2="187.96" y2="45.72" width="0.1524" layer="91"/>
+<label x="185.42" y="45.72" size="1.778" layer="95" rot="MR0"/>
+</segment>
+<segment>
 <pinref part="X1" gate="G$1" pin="GPIO5"/>
 <label x="104.14" y="73.66" size="1.778" layer="95"/>
 <wire x1="121.92" y1="73.66" x2="101.6" y2="73.66" width="0.1524" layer="91"/>
 </segment>
-<segment>
-<wire x1="83.82" y1="111.76" x2="81.28" y2="111.76" width="0.1524" layer="91"/>
-<label x="83.82" y="111.76" size="1.778" layer="95"/>
-<pinref part="J5" gate="G$1" pin="3"/>
-</segment>
-<segment>
-<pinref part="IC1" gate="G$1" pin="SDA"/>
-<wire x1="185.42" y1="43.18" x2="187.96" y2="43.18" width="0.1524" layer="91"/>
-<label x="185.42" y="43.18" size="1.778" layer="95" rot="MR0"/>
-</segment>
-</net>
-<net name="SCL" class="0">
-<segment>
-<pinref part="X1" gate="G$1" pin="GPIO0"/>
-<label x="104.14" y="71.12" size="1.778" layer="95"/>
-<wire x1="101.6" y1="71.12" x2="121.92" y2="71.12" width="0.1524" layer="91"/>
-</segment>
-<segment>
-<wire x1="83.82" y1="114.3" x2="81.28" y2="114.3" width="0.1524" layer="91"/>
-<label x="83.82" y="114.3" size="1.778" layer="95"/>
-<pinref part="J5" gate="G$1" pin="4"/>
-</segment>
-<segment>
-<pinref part="IC1" gate="G$1" pin="SCL"/>
-<wire x1="185.42" y1="45.72" x2="187.96" y2="45.72" width="0.1524" layer="91"/>
-<label x="185.42" y="45.72" size="1.778" layer="95" rot="MR0"/>
-</segment>
-<segment>
-<pinref part="SW8" gate="G$1" pin="P$2"/>
-<label x="137.16" y="152.4" size="1.778" layer="95"/>
-<wire x1="132.08" y1="154.94" x2="132.08" y2="152.4" width="0.1524" layer="91"/>
-<wire x1="132.08" y1="152.4" x2="132.08" y2="149.86" width="0.1524" layer="91"/>
-<wire x1="137.16" y1="152.4" x2="132.08" y2="152.4" width="0.1524" layer="91"/>
-<pinref part="R5" gate="G$1" pin="1"/>
-</segment>
 </net>
 <net name="UART_TX" class="0">
@@
 </segment>
 </net>
-<net name="GPIO16" class="0">
-<segment>
-<pinref part="X1" gate="G$1" pin="GPIO16"/>
-<wire x1="66.04" y1="73.66" x2="45.72" y2="73.66" width="0.1524" layer="91"/>
-<label x="63.5" y="73.66" size="1.778" layer="95" rot="MR0"/>
-</segment>
-</net>
 <net name="SCK" class="0">
 <segment>
@@
 <wire x1="251.46" y1="104.14" x2="256.54" y2="104.14" width="0.1524" layer="91"/>
 <label x="256.54" y="104.14" size="1.778" layer="95"/>
-</segment>
-</net>
-<net name="GPIO4" class="0">
-<segment>
-<pinref part="X1" gate="G$1" pin="GPIO4"/>
-<wire x1="101.6" y1="76.2" x2="121.92" y2="76.2" width="0.1524" layer="91"/>
-<label x="104.14" y="76.2" size="1.778" layer="95"/>
 </segment>
 </net>
@@
 <label x="185.42" y="111.76" size="1.778" layer="95" rot="MR0"/>
 </segment>
+<segment>
+<pinref part="X1" gate="G$1" pin="GPIO16"/>
+<wire x1="66.04" y1="73.66" x2="45.72" y2="73.66" width="0.1524" layer="91"/>
+<label x="63.5" y="73.66" size="1.778" layer="95" rot="MR0"/>
+</segment>
 </net>
 <net name="TFT_DC" class="0">
@@
 </segment>
 </net>
+<net name="GPIO0" class="0">
+<segment>
+<pinref part="X1" gate="G$1" pin="GPIO0"/>
+<label x="104.14" y="71.12" size="1.778" layer="95"/>
+<wire x1="101.6" y1="71.12" x2="121.92" y2="71.12" width="0.1524" layer="91"/>
+</segment>
+<segment>
+<pinref part="SW8" gate="G$1" pin="P$2"/>
+<label x="137.16" y="152.4" size="1.778" layer="95"/>
+<wire x1="132.08" y1="154.94" x2="132.08" y2="152.4" width="0.1524" layer="91"/>
+<wire x1="132.08" y1="152.4" x2="132.08" y2="149.86" width="0.1524" layer="91"/>
+<wire x1="137.16" y1="152.4" x2="132.08" y2="152.4" width="0.1524" layer="91"/>
+<pinref part="R5" gate="G$1" pin="1"/>
+</segment>
+</net>
