File: board/Dilbert-Badge.sch (EAGLE design)
At the start: 31 parts, among them IC1 MCP23017SO, J5 I2C, J6 UART, J7 NEOPIXEL, SW1 UP, SW2 DOWN, SW3 LEFT, SW4 RIGHT, SW5 A, SW6 B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

Commit message: board updates
Parts:
- removed J6: UART, SparkFun-Connectors:M06SILK_FEMALE_PTH
- added J2: FTDI_DEVICE, SparkFun-Connectors:FTDI_DEVICE
- added JP1, JP2, JP3: JUMPER-PAD-3-NOFULL_BOX_SILK, SparkFun-Passives:JUMPER-PAD-3-NOFULL_BOX_SILK
- added JP4, JP5: JUMPER-PAD-2-NC_BY_TRACENO_SILK, SparkFun-Passives:JUMPER-PAD-2-NC_BY_TRACENO_SILK
- added R4: 10K, adafruit:R-US_R0805
Connections:
- new net MCP_IO_A0: IC1.A0, JP1.2
- new net MCP_IO_A1: IC1.A1, JP2.2
- new net MCP_IO_A2: IC1.A2, JP3.2
- new net MCP_IO_INT: IC1.INTA, JP4.2
- new net MCP_IO_RST: IC1.!RESET, R4.1
- net 3V3: now also J2.VCC, JP1.3, JP2.3, JP3.3, R4.2; no longer J6.4
- net GND: now also J2.GND, JP1.1, JP2.1, JP3.1; no longer J6.6
- net SD_CS: now also JP5.2
- net UART_CTS: now also J2.CTS; no longer J6.5
- net UART_DTR: now also J2.DTR; no longer J6.1
- net UART_RX: now also J2.RXI, JP5.1; no longer J6.3
- net UART_TX: now also J2.TXO, JP4.1; no longer J6.2
Changed lines of the file:
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@@
 <setting verticaltext="up"/>
 </settings>
-<grid distance="0.1" unitdist="inch" unit="inch" style="lines" multiple="1" display="no" altdistance="0.01" altunitdist="inch" altunit="inch"/>
+<grid distance="0.1" unitdist="inch" unit="inch" style="lines" multiple="1" display="yes" altdistance="0.01" altunitdist="inch" altunit="inch"/>
 <layers>
 <layer number="1" name="Top" color="4" fill="1" visible="no" active="no"/>
@@
 <part name="J7" library="connectors" deviceset="3X1_SMD_HEADER" device="" value="NEOPIXEL"/>
 <part name="J5" library="SparkFun-Connectors" deviceset="M04" device="PTH" value="I2C"/>
-<part name="J6" library="SparkFun-Connectors" deviceset="M06" device="SILK_FEMALE_PTH" value="UART"/>
 <part name="J1" library="connectors" deviceset="10X1_SMD_HEADER" device=""/>
 <part name="LED5" library="adafruit" deviceset="WS2812B" device="5050"/>
@@
 <part name="LED7" library="adafruit" deviceset="WS2812B" device="5050"/>
 <part name="LED8" library="adafruit" deviceset="WS2812B" device="5050"/>
+<part name="R4" library="adafruit" deviceset="R-US_" device="R0805" value="10K"/>
+<part name="J2" library="SparkFun-Connectors" deviceset="FTDI_DEVICE" device=""/>
+<part name="JP1" library="SparkFun-Passives" deviceset="JUMPER-PAD-3-NO" device="FULL_BOX_SILK"/>
+<part name="JP2" library="SparkFun-Passives" deviceset="JUMPER-PAD-3-NO" device="FULL_BOX_SILK"/>
+<part name="JP3" library="SparkFun-Passives" deviceset="JUMPER-PAD-3-NO" device="FULL_BOX_SILK"/>
+<part name="JP4" library="SparkFun-Passives" deviceset="JUMPER-PAD-2-NC_BY_TRACE" device="NO_SILK"/>
+<part name="JP5" library="SparkFun-Passives" deviceset="JUMPER-PAD-2-NC_BY_TRACE" device="NO_SILK"/>
 </parts>
 <sheets>
@@
 <instance part="J7" gate="G$1" x="104.14" y="106.68"/>
 <instance part="J5" gate="G$1" x="76.2" y="109.22"/>
-<instance part="J6" gate="G$1" x="40.64" y="111.76"/>
 <instance part="J1" gate="G$1" x="99.06" y="210.82" rot="R180"/>
 <instance part="LED5" gate="G$1" x="165.1" y="38.1"/>
@@
 <instance part="LED7" gate="G$1" x="220.98" y="38.1"/>
 <instance part="LED8" gate="G$1" x="248.92" y="38.1"/>
+<instance part="R4" gate="G$1" x="233.68" y="144.78" rot="R90"/>
+<instance part="J2" gate="G$1" x="40.64" y="111.76" rot="R180"/>
+<instance part="JP1" gate="G$1" x="162.56" y="231.14" rot="R180"/>
+<instance part="JP2" gate="G$1" x="162.56" y="213.36" rot="R180"/>
+<instance part="JP3" gate="G$1" x="162.56" y="195.58" rot="R180"/>
+<instance part="JP4" gate="G$1" x="220.98" y="231.14"/>
+<instance part="JP5" gate="G$1" x="220.98" y="213.36"/>
 </instances>
 <busses>
@@
 <wire x1="48.26" y1="119.38" x2="45.72" y2="119.38" width="0.1524" layer="91"/>
 <label x="48.26" y="119.38" size="1.778" layer="95"/>
-<pinref part="J6" gate="G$1" pin="6"/>
+<pinref part="J2" gate="G$1" pin="GND"/>
 </segment>
 <segment>
@@
 <wire x1="251.46" y1="27.94" x2="248.92" y2="27.94" width="0.1524" layer="91"/>
 <label x="251.46" y="27.94" size="1.778" layer="95"/>
+</segment>
+<segment>
+<pinref part="JP1" gate="G$1" pin="1"/>
+<wire x1="162.56" y1="226.06" x2="165.1" y2="226.06" width="0.1524" layer="91"/>
+<label x="165.1" y="226.06" size="1.778" layer="95"/>
+</segment>
+<segment>
+<pinref part="JP3" gate="G$1" pin="1"/>
+<wire x1="162.56" y1="190.5" x2="165.1" y2="190.5" width="0.1524" layer="91"/>
+<label x="165.1" y="190.5" size="1.778" layer="95"/>
+</segment>
+<segment>
+<pinref part="JP2" gate="G$1" pin="1"/>
+<wire x1="162.56" y1="208.28" x2="165.1" y2="208.28" width="0.1524" layer="91"/>
+<label x="165.1" y="208.28" size="1.778" layer="95"/>
 </segment>
 </net>
@@
 <wire x1="45.72" y1="109.22" x2="48.26" y2="109.22" width="0.1524" layer="91"/>
 <label x="48.26" y="109.22" size="1.778" layer="95"/>
-<pinref part="J6" gate="G$1" pin="2"/>
+<pinref part="J2" gate="G$1" pin="TXO"/>
+</segment>
+<segment>
+<pinref part="JP4" gate="G$1" pin="1"/>
+<wire x1="213.36" y1="231.14" x2="215.9" y2="231.14" width="0.1524" layer="91"/>
+<label x="213.36" y="231.14" size="1.778" layer="95" rot="MR0"/>
 </segment>
 </net>
@@
 <wire x1="45.72" y1="111.76" x2="48.26" y2="111.76" width="0.1524" layer="91"/>
 <label x="48.26" y="111.76" size="1.778" layer="95"/>
-<pinref part="J6" gate="G$1" pin="3"/>
+<pinref part="J2" gate="G$1" pin="RXI"/>
+</segment>
+<segment>
+<pinref part="JP5" gate="G$1" pin="1"/>
+<wire x1="213.36" y1="213.36" x2="215.9" y2="213.36" width="0.1524" layer="91"/>
+<label x="213.36" y="213.36" size="1.778" layer="95" rot="MR0"/>
 </segment>
 </net>
@@
 <wire x1="45.72" y1="116.84" x2="48.26" y2="116.84" width="0.1524" layer="91"/>
 <label x="48.26" y="116.84" size="1.778" layer="95"/>
-<pinref part="J6" gate="G$1" pin="5"/>
+<pinref part="J2" gate="G$1" pin="CTS"/>
 </segment>
 </net>
@@
 <wire x1="45.72" y1="106.68" x2="48.26" y2="106.68" width="0.1524" layer="91"/>
 <label x="48.26" y="106.68" size="1.778" layer="95"/>
-<pinref part="J6" gate="G$1" pin="1"/>
+<pinref part="J2" gate="G$1" pin="DTR"/>
 </segment>
 </net>
@@
 <wire x1="48.26" y1="114.3" x2="45.72" y2="114.3" width="0.1524" layer="91"/>
 <label x="48.26" y="114.3" size="1.778" layer="95"/>
-<pinref part="J6" gate="G$1" pin="4"/>
+<pinref part="J2" gate="G$1" pin="VCC"/>
 </segment>
 <segment>
@@
 <wire x1="256.54" y1="53.34" x2="254" y2="53.34" width="0.1524" layer="91"/>
 <label x="256.54" y="53.34" size="1.778" layer="95"/>
+</segment>
+<segment>
+<pinref part="JP3" gate="G$1" pin="3"/>
+<wire x1="162.56" y1="200.66" x2="165.1" y2="200.66" width="0.1524" layer="91"/>
+<label x="165.1" y="200.66" size="1.778" layer="95"/>
+</segment>
+<segment>
+<pinref part="JP2" gate="G$1" pin="3"/>
+<wire x1="162.56" y1="218.44" x2="165.1" y2="218.44" width="0.1524" layer="91"/>
+<label x="165.1" y="218.44" size="1.778" layer="95"/>
+</segment>
+<segment>
+<pinref part="JP1" gate="G$1" pin="3"/>
+<wire x1="162.56" y1="236.22" x2="165.1" y2="236.22" width="0.1524" layer="91"/>
+<label x="165.1" y="236.22" size="1.778" layer="95"/>
+</segment>
+<segment>
+<pinref part="R4" gate="G$1" pin="2"/>
+<wire x1="233.68" y1="154.94" x2="233.68" y2="149.86" width="0.1524" layer="91"/>
+<label x="233.68" y="154.94" size="1.778" layer="95"/>
 </segment>
 </net>
@@
 <label x="254" y="83.82" size="1.778" layer="95"/>
 </segment>
+<segment>
+<pinref part="JP5" gate="G$1" pin="2"/>
+<wire x1="226.06" y1="213.36" x2="228.6" y2="213.36" width="0.1524" layer="91"/>
+<label x="228.6" y="213.36" size="1.778" layer="95"/>
+</segment>
 </net>
 <net name="N$4" class="0">
@@
 </segment>
 </net>
+<net name="MCP_IO_A0" class="0">
+<segment>
+<pinref part="IC1" gate="G$1" pin="A0"/>
+<wire x1="45.72" y1="203.2" x2="48.26" y2="203.2" width="0.1524" layer="91"/>
+<label x="45.72" y="203.2" size="1.778" layer="95" rot="MR0"/>
+</segment>
+<segment>
+<pinref part="JP1" gate="G$1" pin="2"/>
+<wire x1="167.64" y1="231.14" x2="170.18" y2="231.14" width="0.1524" layer="91"/>
+<label x="170.18" y="231.14" size="1.778" layer="95"/>
+</segment>
+</net>
+<net name="MCP_IO_A1" class="0">
+<segment>
+<pinref part="IC1" gate="G$1" pin="A1"/>
+<wire x1="45.72" y1="200.66" x2="48.26" y2="200.66" width="0.1524" layer="91"/>
+<label x="45.72" y="200.66" size="1.778" layer="95" rot="MR0"/>
+</segment>
+<segment>
+<pinref part="JP2" gate="G$1" pin="2"/>
+<wire x1="167.64" y1="213.36" x2="170.18" y2="213.36" width="0.1524" layer="91"/>
+<label x="170.18" y="213.36" size="1.778" layer="95"/>
+</segment>
+</net>
+<net name="MCP_IO_A2" class="0">
+<segment>
+<pinref part="IC1" gate="G$1" pin="A2"/>
+<wire x1="45.72" y1="198.12" x2="48.26" y2="198.12" width="0.1524" layer="91"/>
+<label x="45.72" y="198.12" size="1.778" layer="95" rot="MR0"/>
+</segment>
+<segment>
+<pinref part="JP3" gate="G$1" pin="2"/>
+<wire x1="167.64" y1="195.58" x2="170.18" y2="195.58" width="0.1524" layer="91"/>
+<label x="170.18" y="195.58" size="1.778" layer="95"/>
+</segment>
+</net>
+<net name="MCP_IO_RST" class="0">
+<segment>
+<pinref part="IC1" gate="G$1" pin="!RESET"/>
+<wire x1="45.72" y1="228.6" x2="48.26" y2="228.6" width="0.1524" layer="91"/>
+<label x="45.72" y="228.6" size="1.778" layer="95" rot="MR0"/>
+</segment>
+<segment>
+<pinref part="R4" gate="G$1" pin="1"/>
+<wire x1="233.68" y1="139.7" x2="233.68" y2="134.62" width="0.1524" layer="91"/>
+<label x="233.68" y="134.62" size="1.778" layer="95" rot="MR180"/>
+</segment>
+</net>
+<net name="MCP_IO_INT" class="0">
+<segment>
+<pinref part="IC1" gate="G$1" pin="INTA"/>
+<wire x1="45.72" y1="223.52" x2="48.26" y2="223.52" width="0.1524" layer="91"/>
+<label x="45.72" y="223.52" size="1.778" layer="95" rot="MR0"/>
+</segment>
+<segment>
+<pinref part="JP4" gate="G$1" pin="2"/>
+<wire x1="226.06" y1="231.14" x2="228.6" y2="231.14" width="0.1524" layer="91"/>
+<label x="228.6" y="231.14" size="1.778" layer="95"/>
+</segment>
+</net>

Commit message: more board layout
Parts:
- removed J7: NEOPIXEL, connectors:3X1_SMD_HEADER
- added J3: NEOPIXEL, SparkFun-Connectors:M03PTH
- added U$2, U$3: 5MM_MOUNTING_HOLE, mechanical:5MM_MOUNTING_HOLE
- J1: value (none) -> IO EXP.; device connectors:10X1_SMD_HEADER -> SparkFun-Connectors:M10SILK_FEMALE_PTH
- JP1: value JUMPER-PAD-3-NOFULL_BOX_SILK -> MCP IO A0; device SparkFun-Passives:JUMPER-PAD-3-NOFULL_BOX_SILK -> SparkFun-Passives:JUMPER-PAD-3-NOYES_SILK
- JP2: value JUMPER-PAD-3-NOFULL_BOX_SILK -> MCP IO A1; device SparkFun-Passives:JUMPER-PAD-3-NOFULL_BOX_SILK -> SparkFun-Passives:JUMPER-PAD-3-NOYES_SILK
- JP3: value JUMPER-PAD-3-NOFULL_BOX_SILK -> MCP IO A2; device SparkFun-Passives:JUMPER-PAD-3-NOFULL_BOX_SILK -> SparkFun-Passives:JUMPER-PAD-3-NOYES_SILK
- JP4: value JUMPER-PAD-2-NC_BY_TRACENO_SILK -> IO INT TO UART TX
- JP5: value JUMPER-PAD-2-NC_BY_TRACENO_SILK -> SD CS TO UART RX
Connections:
- net 3V3: now also J3.2; no longer J7.2
- net GND: now also J3.1; no longer J7.1
- net NEOPIXEL_OUT: now also J3.3; no longer J7.3
Changed lines of the file:
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@@
 <part name="U$1" library="displays" deviceset="2.2IN_ILI9341" device=""/>
 <part name="R7" library="adafruit" deviceset="R-US_" device="R0805" value="10K"/>
-<part name="J7" library="connectors" deviceset="3X1_SMD_HEADER" device="" value="NEOPIXEL"/>
 <part name="J5" library="SparkFun-Connectors" deviceset="M04" device="PTH" value="I2C"/>
-<part name="J1" library="connectors" deviceset="10X1_SMD_HEADER" device=""/>
 <part name="LED5" library="adafruit" deviceset="WS2812B" device="5050"/>
 <part name="LED6" library="adafruit" deviceset="WS2812B" device="5050"/>
@@
 <part name="R4" library="adafruit" deviceset="R-US_" device="R0805" value="10K"/>
 <part name="J2" library="SparkFun-Connectors" deviceset="FTDI_DEVICE" device=""/>
-<part name="JP1" library="SparkFun-Passives" deviceset="JUMPER-PAD-3-NO" device="FULL_BOX_SILK"/>
-<part name="JP2" library="SparkFun-Passives" deviceset="JUMPER-PAD-3-NO" device="FULL_BOX_SILK"/>
-<part name="JP3" library="SparkFun-Passives" deviceset="JUMPER-PAD-3-NO" device="FULL_BOX_SILK"/>
-<part name="JP4" library="SparkFun-Passives" deviceset="JUMPER-PAD-2-NC_BY_TRACE" device="NO_SILK"/>
-<part name="JP5" library="SparkFun-Passives" deviceset="JUMPER-PAD-2-NC_BY_TRACE" device="NO_SILK"/>
+<part name="JP1" library="SparkFun-Passives" deviceset="JUMPER-PAD-3-NO" device="YES_SILK" value="MCP IO A0"/>
+<part name="JP2" library="SparkFun-Passives" deviceset="JUMPER-PAD-3-NO" device="YES_SILK" value="MCP IO A1"/>
+<part name="JP3" library="SparkFun-Passives" deviceset="JUMPER-PAD-3-NO" device="YES_SILK" value="MCP IO A2"/>
+<part name="JP4" library="SparkFun-Passives" deviceset="JUMPER-PAD-2-NC_BY_TRACE" device="NO_SILK" value="IO INT TO UART TX"/>
+<part name="JP5" library="SparkFun-Passives" deviceset="JUMPER-PAD-2-NC_BY_TRACE" device="NO_SILK" value="SD CS TO UART RX"/>
+<part name="U$2" library="mechanical" deviceset="5MM_MOUNTING_HOLE" device=""/>
+<part name="U$3" library="mechanical" deviceset="5MM_MOUNTING_HOLE" device=""/>
+<part name="J1" library="SparkFun-Connectors" deviceset="M10" device="SILK_FEMALE_PTH" value="IO EXP."/>
+<part name="J3" library="SparkFun-Connectors" deviceset="M03" device="PTH" value="NEOPIXEL"/>
 </parts>
 <sheets>
@@
 <instance part="U$1" gate="G$1" x="218.44" y="88.9"/>
 <instance part="R7" gate="G$1" x="210.82" y="144.78" rot="R90"/>
-<instance part="J7" gate="G$1" x="104.14" y="106.68"/>
 <instance part="J5" gate="G$1" x="76.2" y="109.22"/>
-<instance part="J1" gate="G$1" x="99.06" y="210.82" rot="R180"/>
 <instance part="LED5" gate="G$1" x="165.1" y="38.1"/>
 <instance part="LED6" gate="G$1" x="193.04" y="38.1"/>
@@
 <instance part="JP4" gate="G$1" x="220.98" y="231.14"/>
 <instance part="JP5" gate="G$1" x="220.98" y="213.36"/>
+<instance part="U$2" gate="G$1" x="35.56" y="10.16"/>
+<instance part="U$3" gate="G$1" x="50.8" y="10.16"/>
+<instance part="J1" gate="G$1" x="104.14" y="193.04" rot="R180"/>
+<instance part="J3" gate="J$1" x="101.6" y="109.22"/>
 </instances>
 <busses>
@@
 <wire x1="111.76" y1="106.68" x2="109.22" y2="106.68" width="0.1524" layer="91"/>
 <label x="111.76" y="106.68" size="1.778" layer="95"/>
-<pinref part="J7" gate="G$1" pin="1"/>
+<pinref part="J3" gate="J$1" pin="1"/>
 </segment>
 <segment>
@@
 <wire x1="111.76" y1="111.76" x2="109.22" y2="111.76" width="0.1524" layer="91"/>
 <label x="111.76" y="111.76" size="1.778" layer="95"/>
-<pinref part="J7" gate="G$1" pin="3"/>
+<pinref part="J3" gate="J$1" pin="3"/>
 </segment>
 <segment>
@@
 <wire x1="111.76" y1="109.22" x2="109.22" y2="109.22" width="0.1524" layer="91"/>
 <label x="111.76" y="109.22" size="1.778" layer="95"/>
-<pinref part="J7" gate="G$1" pin="2"/>
+<pinref part="J3" gate="J$1" pin="2"/>
 </segment>
 <segment>
@@
 <segment>
 <pinref part="IC1" gate="G$1" pin="GPB0"/>
+<wire x1="73.66" y1="210.82" x2="93.98" y2="210.82" width="0.1524" layer="91"/>
 <pinref part="J1" gate="G$1" pin="1"/>
-<wire x1="73.66" y1="210.82" x2="93.98" y2="210.82" width="0.1524" layer="91"/>
 </segment>
 </net>
 <net name="N$5" class="0">
 <segment>
-<pinref part="J1" gate="G$1" pin="2"/>
 <pinref part="IC1" gate="G$1" pin="GPB1"/>
 <wire x1="93.98" y1="208.28" x2="73.66" y2="208.28" width="0.1524" layer="91"/>
+<pinref part="J1" gate="G$1" pin="2"/>
 </segment>
 </net>
@@
 <segment>
 <pinref part="IC1" gate="G$1" pin="GPB2"/>
+<wire x1="73.66" y1="205.74" x2="93.98" y2="205.74" width="0.1524" layer="91"/>
 <pinref part="J1" gate="G$1" pin="3"/>
-<wire x1="73.66" y1="205.74" x2="93.98" y2="205.74" width="0.1524" layer="91"/>
 </segment>
 </net>
 <net name="N$7" class="0">
 <segment>
-<pinref part="J1" gate="G$1" pin="4"/>
 <pinref part="IC1" gate="G$1" pin="GPB3"/>
 <wire x1="93.98" y1="203.2" x2="73.66" y2="203.2" width="0.1524" layer="91"/>
+<pinref part="J1" gate="G$1" pin="4"/>
 </segment>
 </net>
@@
 <wire x1="73.66" y1="215.9" x2="81.28" y2="215.9" width="0.1524" layer="91"/>
 <wire x1="81.28" y1="215.9" x2="81.28" y2="187.96" width="0.1524" layer="91"/>
+<wire x1="81.28" y1="187.96" x2="93.98" y2="187.96" width="0.1524" layer="91"/>
 <pinref part="J1" gate="G$1" pin="10"/>
-<wire x1="81.28" y1="187.96" x2="93.98" y2="187.96" width="0.1524" layer="91"/>
 </segment>
 </net>
 <net name="N$9" class="0">
 <segment>
-<pinref part="J1" gate="G$1" pin="9"/>
 <wire x1="93.98" y1="190.5" x2="83.82" y2="190.5" width="0.1524" layer="91"/>
 <wire x1="83.82" y1="190.5" x2="83.82" y2="218.44" width="0.1524" layer="91"/>
 <pinref part="IC1" gate="G$1" pin="GPA6"/>
 <wire x1="83.82" y1="218.44" x2="73.66" y2="218.44" width="0.1524" layer="91"/>
+<pinref part="J1" gate="G$1" pin="9"/>
 </segment>
 </net>
@@
 <segment>
 <pinref part="IC1" gate="G$1" pin="GPB7"/>
+<wire x1="73.66" y1="193.04" x2="93.98" y2="193.04" width="0.1524" layer="91"/>
 <pinref part="J1" gate="G$1" pin="8"/>
-<wire x1="73.66" y1="193.04" x2="93.98" y2="193.04" width="0.1524" layer="91"/>
 </segment>
 </net>
 <net name="N$11" class="0">
 <segment>
-<pinref part="J1" gate="G$1" pin="7"/>
 <pinref part="IC1" gate="G$1" pin="GPB6"/>
 <wire x1="93.98" y1="195.58" x2="73.66" y2="195.58" width="0.1524" layer="91"/>
+<pinref part="J1" gate="G$1" pin="7"/>
 </segment>
 </net>
@@
 <segment>
 <pinref part="IC1" gate="G$1" pin="GPB5"/>
+<wire x1="73.66" y1="198.12" x2="93.98" y2="198.12" width="0.1524" layer="91"/>
 <pinref part="J1" gate="G$1" pin="6"/>
-<wire x1="73.66" y1="198.12" x2="93.98" y2="198.12" width="0.1524" layer="91"/>
 </segment>
 </net>
 <net name="N$13" class="0">
 <segment>
-<pinref part="J1" gate="G$1" pin="5"/>
 <pinref part="IC1" gate="G$1" pin="GPB4"/>
 <wire x1="93.98" y1="200.66" x2="73.66" y2="200.66" width="0.1524" layer="91"/>
-</segment>
-</net>
+<pinref part="J1" gate="G$1" pin="5"/>
+</segment>
+</net>
